Commit message: Add files via upload

File: my_vehicle.urdf (robot description, URDF)
Before this commit: robot visual, 5 links, 4 joints
Joints:
- joint left_back_wheel_joint: axis 0 1 0 -> 0 0 1
- joint left_front_wheel_joint: axis 0 1 0 -> 0 0 1
- joint right_back_wheel_joint: axis 0 1 0 -> 0 0 1
- joint right_front_wheel_joint: axis 0 1 0 -> 0 0 1

Commit message: Add files via upload

File: my_vehicle.urdf (robot description, URDF)
Before this commit: robot visual, 5 links, 4 joints
Joints:
- joint left_back_wheel_joint: limit lower=0.0 upper=0.548 effort=1000.0 velocity=0.5 -> (none); type revolute -> continuous
- joint left_front_wheel_joint: limit lower=0.0 upper=0.548 effort=1000.0 velocity=0.5 -> (none); type revolute -> continuous
- joint right_back_wheel_joint: limit lower=0.0 upper=0.548 effort=1000.0 velocity=0.5 -> (none); type revolute -> continuous
- joint right_front_wheel_joint: limit lower=0.0 upper=0.548 effort=1000.0 velocity=0.5 -> (none); type revolute -> continuous
